Commit message: updating fixed joint to world

File: examplerobot_description/urdf/examplerobot.xacro (robot description, xacro)
@@ -81,4 +81,5 @@
            parent="base_link" child="ref_link" />
   -->
+   <link name="world"/>
    <xacro:ref_joint name="world__${link_00_name}" type="fixed"
            axis_xyz="0 0 1"

Commit message: updating fixed joint to world

File: examplerobot_description/urdf/examplerobot.xacro (robot description, xacro)
@@ -74,16 +74,14 @@
               meshfile="package://examplerobot_description/meshes/end_effector.stl"
               meshscale="0.001 0.001 0.001" />
+  <link name="world"/>
+  <xacro:ref_joint name="world__${link_ref_name}" type="fixed"
+           axis_xyz="0 0 1"
+           origin_rpy="0 0 0" origin_xyz="0 0 0"
+           parent="world" child="ref_link" />
   <!-- Joint 0 - ref_link__base_link -->
-  <!--
   <xacro:ref_joint name="${link_ref_name}__${link_00_name}" type="fixed"
            axis_xyz="0 0 1"
            origin_rpy="0 0 0" origin_xyz="0 0 0"
            parent="base_link" child="ref_link" />
-  -->
-   <link name="world"/>
-   <xacro:ref_joint name="world__${link_00_name}" type="fixed"
-           axis_xyz="0 0 1"
-           origin_rpy="0 0 0" origin_xyz="0 0 0"
-           parent="world" child="base_link" />
   <!-- Joint 1 - base_link__link_01 -->
   <xacro:rev_joint name="${link_00_name}__${link_01_name}" type="revolute"

Commit message: adding link6 to URDF

File: examplerobot_description/urdf/examplerobot.xacro (robot description, xacro)
@@ -60,6 +60,15 @@
               meshfile="package://examplerobot_description/meshes/link5.stl"
               meshscale="0.001 0.001 0.001" />
-  <!-- Link 6 - end_effector -->
+  <!-- Link 6 - link_06 -->
   <xacro:link_mesh name="${link_06_name}"
+              origin_rpy="0 0 0" origin_xyz="0 0 0"
+              mass="1.0"
+              ixx="1.3235" ixy="0" ixz="0"
+              iyy="1.3235" iyz="0"
+              izz="0.9655"
+              meshfile="package://examplerobot_description/meshes/link6.stl"
+              meshscale="0.001 0.001 0.001" />
+  <!-- Link 7 - end_effector -->
+  <xacro:link_mesh name="${link_07_name}"
               origin_rpy="0 0 0" origin_xyz="0 0 0"
               mass="1.0"
@@ -123,4 +132,9 @@
            parent="link_05" child="end_effector"
            limit_e="1000" limit_l="-3.14" limit_u="3.14" limit_v="0.5" />
+  <!-- Joint 7 - link_06__end_effector -->
+  <xacro:ref_joint name="${link_ref_name}__${link_00_name}" type="fixed"
+           axis_xyz="0 0 1"
+           origin_rpy="0 0 0" origin_xyz="0 0 0"
+           parent="link_06" child="end_effector" />
   <!-- END - Robot description -->
   <gazebo>

File: examplerobot_description/urdf/robot-parameters.xacro (robot description, xacro)
@@ -8,4 +8,5 @@
   <xacro:property name="link_04_name" value="link_04" />
   <xacro:property name="link_05_name" value="link_05" />
-  <xacro:property name="link_06_name" value="end_effector" />
+  <xacro:property name="link_06_name" value="link_06" />
+  <xacro:property name="link_07_name" value="end_effector" />
 </robot>

Commit message: adding link6 to URDF

File: examplerobot_description/urdf/examplerobot.xacro (robot description, xacro)
@@ -92,5 +92,5 @@
               meshfile="package://examplerobot_description/meshes/base_link.stl"
               meshscale="0.0001 0.0001 0.0001" />
-  <xacro:ref_joint name="${link_ref_name}__${link_00_name}" type="fixed"
+  <xacro:fixed_joint name="${link_ref_name}__${link_00_name}" type="fixed"
            axis_xyz="0 0 1"
            origin_rpy="0 0 0" origin_xyz="0 0 0"
@@ -133,5 +133,5 @@
            limit_e="1000" limit_l="-3.14" limit_u="3.14" limit_v="0.5" />
   <!-- Joint 7 - link_06__end_effector -->
-  <xacro:ref_joint name="${link_06_name}__${link_07_name}" type="fixed"
+  <xacro:fixed_joint name="${link_06_name}__${link_07_name}" type="fixed"
            axis_xyz="0 0 1"
            origin_rpy="0 0 0" origin_xyz="0 0 0"

File: examplerobot_description/urdf/links-joints.xacro (robot description, xacro)
@@ -1,5 +1,5 @@
 <?xml version="1.0" ?>
 <robot xmlns:xacro="http://www.ros.org/wiki/xacro">
-  <xacro:macro name="ref_joint" params="name type axis_xyz origin_rpy origin_xyz parent child ">
+  <xacro:macro name="fixed_joint" params="name type axis_xyz origin_rpy origin_xyz parent child ">
     <joint name="${name}" type="${type}">
       <axis xyz="${axis_xyz}" />

Commit message: realized URDF tag <dh> is not real

File: examplerobot_description/urdf/examplerobot.xacro (robot description, xacro)
@@ -102,4 +102,5 @@
            parent="base_link" child="link_01"
            limit_e="1000" limit_l="-3.14" limit_u="3.14" limit_v="0.5" />
+           <!-- ai="0" di=".350" alphai="-1.571" thetai="0"/> -->
   <!-- Joint 2 - link_01__link02 -->
   <xacro:rev_joint name="${link_01_name}__${link_02_name}" type="revolute"

File: examplerobot_description/urdf/links-joints.xacro (robot description, xacro)
@@ -9,5 +9,5 @@
     </joint>
   </xacro:macro>
-  <xacro:macro name="rev_joint" params="name type axis_xyz origin_rpy origin_xyz parent child limit_e limit_l limit_u limit_v">
+  <xacro:macro name="rev_joint" params="name type axis_xyz origin_rpy origin_xyz parent child limit_e limit_l limit_u limit_v "> <!--ai alphai di "> -->
     <joint name="${name}" type="${type}">
       <axis xyz="${axis_xyz}" />
@@ -20,5 +20,5 @@
         <dynamics damping="0.1" friction="0.1"/>
       </kinematic>
-      <dh param="0.0" a="0.0" alpha="0.0" d="0.0" theta="0.0" />
+      <ddasda!!sdh param="0.0" a="0.0" alpha="0.0" d="0.0" theta="0.0" />
     </joint>
     <transmission name="trans_${name}">
