Commit message: testing </dh> tag, influence not evident

File: examplerobot_description/urdf/links-joints.xacro (robot description, xacro)
@@ -16,4 +16,9 @@
       <parent link="${parent}" />
       <child link="${child}" />
+      <kinematic>
+        <limits effort="100" lower="-3.14" upper="3.14" velocity="1"/>
+        <dynamics damping="0.1" friction="0.1"/>
+      </kinematic>
+      <dh param="0.0" a="0.0" alpha="0.0" d="0.0" theta="0.0" />
     </joint>
     <transmission name="trans_${name}">

Commit message: testing examplerobot-gazebo

File: examplerobot_description/urdf/links-joints.xacro (robot description, xacro)
@@ -16,9 +16,4 @@
       <parent link="${parent}" />
       <child link="${child}" />
-      <kinematic>
-        <limits effort="100" lower="-3.14" upper="3.14" velocity="1"/>
-        <dynamics damping="0.1" friction="0.1"/>
-      </kinematic>
-      <ddasda!!sdh param="0.0" a="0.0" alpha="0.0" d="0.0" theta="0.0" />
     </joint>
     <transmission name="trans_${name}">
